File: prac3/prac3.kicad_pcb (KiCad board)
At the start: 2 copper layers, 47 x 35 mm, 7 parts, among them J1 Screw_Terminal_01x07, SW1 SW_Push

Commit message: prac3 2do parcial
Parts:
- removed the G*** at (81.0, 89.0)
- removed R2: 220, Resistor_SMD:R_0805_2012Metric
- removed REF**: KiCad-Logo2_5mm_SilkScreen, Symbol:KiCad-Logo2_5mm_SilkScreen
- removed SW1: SW_Push, Button_Switch_SMD:SW_Push_1P1T_NO_CK_KMR2
- added BZ1: Buzzer, Buzzer_Beeper:Buzzer_15x7.5RM7.6, F.Cu at (148.0, 79.2)
- added G***: LOGO, logos:logo_drilo, F.Cu at (160.5, 77.0)
- added J2: Conn_01x03_Pin, Connector_PinHeader_2.54mm:PinHeader_1x03_P2.54mm_Vertical, F.Cu at (134.5, 93.9)
- added U1: LM35-LP, Package_TO_SOT_THT:TO-92_Inline, F.Cu at (151.9, 95.8)
- J1: value Screw_Terminal_01x07 -> Conn_01x02_Pin; footprint TerminalBlock_Phoenix:TerminalBlock_Phoenix_MKDS-1,5-7_1x07_P5.00mm_Horizontal -> Connector_PinHeader_2.54mm:PinHeader_1x02_P2.54mm_Vertical
- R1: value 220 -> R
- moved D1 81.2 mm to (151.5, 101.5), turned to 180 degrees
- moved R1 72.5 mm to (144.4, 100.3), turned to 90 degrees
- moved J1 37.7 mm to (134.5, 83.0), turned to 0 degrees
Connections:
- J1 pad 2: Net-(J1-Pin_2) -> GND
- R1 pad 1: Net-(J1-Pin_6) -> Net-(D1-A)
- R1 pad 2: Net-(D1-A) -> Net-(J2-Pin_3)
Routing:
- net Net-(J1-Pin_3): track 30.3 -> 0.00 mm
- net GND: track 22.3 -> 41.8 mm
- net Net-(J2-Pin_2): track 0.00 -> 17.6 mm
- net Net-(J2-Pin_1): track 0.00 -> 17.6 mm
- net Net-(J1-Pin_6): track 12.2 -> 0.00 mm
- net Net-(J1-Pin_2): track 11.7 -> 0.00 mm
- net Net-(J2-Pin_3): track 0.00 -> 10.0 mm
- net Net-(BZ1-+): track 23.7 -> 15.1 mm
- net Net-(D1-A): track 8.45 -> 6.33 mm
- added copper zone on F.Cu, net (none)
- added copper zone on B.Cu, net GND
- removed copper zone on F.Cu, net GND
Other:
- board size 47 x 35 mm -> 39 x 34 mm
- board text added: "LM32 CON BUZZER"
- board text removed: "CORRIENTE"
- board text removed: "DATOS"
- board text removed: "GND"
