File: prac4/prac4.kicad_pcb (KiCad board)
At the start: 2 copper layers, 7 parts, among them J1 Screw_Terminal_01x04

Commit message: prac 4 2do parcial
prac 4 2do parcial
Parts:
- removed the G*** at (93.0, 115.0)
- removed the REF** at (120.0, 116.0)
- added D2: LED, LED_LTL-4233_LTO:LED_LTL-4233_LTO, F.Cu at (195.6, 112.5)
- added D3: LED, LED_LTL-4233_LTO:LED_LTL-4233_LTO, F.Cu at (195.6, 121.0)
- added G***: LOGO, logos:logo_drilo, F.Cu at (187.0, 124.0)
- added REF**: KiCad-Logo2_5mm_SilkScreen, Symbol:KiCad-Logo2_5mm_SilkScreen, F.Cu at (177.5, 122.0)
- D1: value LED_BRKG -> LED; footprint LED_SMD:LED_RGB_1210 -> LED_LTL-4233_LTO:LED_LTL-4233_LTO
- J1: value Screw_Terminal_01x04 -> OSTVN04A150; footprint TerminalBlock_Phoenix:TerminalBlock_Phoenix_MKDS-1,5-4-5.08_1x04_P5.08mm_Horizontal -> TerminalBlock_OSTVN04A150:TerminalBlock_OSTVN04A150
- moved R2 86.0 mm to (187.0, 113.0)
- moved R3 86.0 mm to (187.0, 118.0)
- moved R1 85.9 mm to (187.0, 107.0)
- moved D1 85.4 mm to (195.5, 105.0), turned to 180 degrees
- moved J1 81.4 mm to (178.0, 107.0), turned to -90 degrees
Connections:
- D1 pad 1: Net-(D1-BA) -> GND
- D1 pad 2: Net-(D1-RA) -> Net-(D1-A)
- J1 pad 1: Net-(J1-Pin_1) -> GND
- J1 pad 2: Net-(J1-Pin_2) -> Net-(J1-Pad2)
- J1 pad 3: Net-(J1-Pin_2) -> Net-(J1-Pad3)
- J1 pad 4: GND -> Net-(J1-Pad4)
- R1 pad 1: Net-(J1-Pin_2) -> Net-(J1-Pad4)
- R1 pad 2: Net-(D1-BA) -> Net-(D1-A)
- R2 pad 1: Net-(J1-Pin_2) -> Net-(J1-Pad3)
- R2 pad 2: Net-(D1-GA) -> Net-(D2-A)
- R3 pad 1: Net-(J1-Pin_1) -> Net-(J1-Pad2)
- R3 pad 2: Net-(D1-RA) -> Net-(D3-A)
Routing:
- net Net-(J1-Pin_2): track 29.3 -> 0.00 mm
- net Net-(J1-Pin_1): track 21.5 -> 0.00 mm
- net GND: track 16.2 -> 37.2 mm
- net Net-(J1-Pad4): track 0.00 -> 14.2 mm, vias 0 -> 2
- net Net-(J1-Pad2): track 0.00 -> 13.7 mm
- net Net-(D1-GA): track 11.4 -> 0.00 mm
- net Net-(D1-BA): track 9.08 -> 0.00 mm, vias 2 -> 0
- net Net-(J1-Pad3): track 0.00 -> 8.93 mm, vias 0 -> 2
- net Net-(D1-RA): track 8.57 -> 0.00 mm
- net Net-(D3-A): track 0.00 -> 8.13 mm
- net Net-(D1-A): track 0.00 -> 7.05 mm
- net Net-(D2-A): track 0.00 -> 5.33 mm
- added copper zone on F.Cu, net GND
Other:
- board outline added: 33 x 29.5 mm
- board text added: "GND"
- board text added: "P_L1"
- board text added: "P_L2"
- board text added: "P_L3"
- board text removed: "Practica 4"
